Commit message: ConfigManager complete, Inertia added

File: src/robco_description/gazebo/robco_gazebo.xacro (robot description, xacro)
@@ -4,6 +4,7 @@
     <!-- ros_control plugin -->
     <gazebo>
-      <plugin filename="gz_ros2_control-system" name="gz_ros2_control::GazeboSimROS2ControlPlugin">
+    <plugin filename="libgazebo_ros2_control.so" name="gazebo_ros2_control">
         <parameters>$(find robco_description)/ros2_control/ros2_controllers.yaml</parameters>
+        <controlPeriod>0.01</controlPeriod>
       </plugin>
     </gazebo>
@@ -98,4 +99,61 @@
       <material>Gazebo/Gray</material>
     </gazebo>
+    <gazebo reference="base__drive1">
+      <preserveFixedJoint>true</preserveFixedJoint>
+    </gazebo>
+    <gazebo reference="drive1__drive1_shaft">
+      <preserveFixedJoint>true</preserveFixedJoint>
+    </gazebo>
+    <gazebo reference="drive1_distal__drive2">
+      <preserveFixedJoint>true</preserveFixedJoint>
+    </gazebo>
+    <gazebo reference="drive2__drive2_shaft">
+      <preserveFixedJoint>true</preserveFixedJoint>
+    </gazebo>
+    <gazebo reference="drive2_distal__link0">
+      <preserveFixedJoint>true</preserveFixedJoint>
+    </gazebo>
+    <gazebo reference="link0__drive3">
+      <preserveFixedJoint>true</preserveFixedJoint>
+    </gazebo>
+    <gazebo reference="drive3__drive3_shaft">
+      <preserveFixedJoint>true</preserveFixedJoint>
+    </gazebo>
+    <gazebo reference="drive3_distal__drive4">
+      <preserveFixedJoint>true</preserveFixedJoint>
+    </gazebo>
+    <gazebo reference="drive4__drive4_shaft">
+      <preserveFixedJoint>true</preserveFixedJoint>
+    </gazebo>
+    <gazebo reference="drive4_distal__link1">
+      <preserveFixedJoint>true</preserveFixedJoint>
+    </gazebo>
+    <gazebo reference="link1__drive5">
+      <preserveFixedJoint>true</preserveFixedJoint>
+    </gazebo>
+    <gazebo reference="drive5__drive5_shaft">
+      <preserveFixedJoint>true</preserveFixedJoint>
+    </gazebo>
+    <gazebo reference="drive5_distal__drive6">
+      <preserveFixedJoint>true</preserveFixedJoint>
+    </gazebo>
+    <gazebo reference="drive6__drive6_shaft">
+      <preserveFixedJoint>true</preserveFixedJoint>
+    </gazebo>
+    <gazebo reference="drive6_distal__robco_handeye">
+      <preserveFixedJoint>true</preserveFixedJoint>
+    </gazebo>
+    <gazebo reference="robco_handeye_flange_joint">
+      <preserveFixedJoint>true</preserveFixedJoint>
+    </gazebo>
+    <gazebo reference="robco_hand_joint">
+      <preserveFixedJoint>true</preserveFixedJoint>
+    </gazebo>
+    <gazebo reference="robco_palmjoint">
+      <preserveFixedJoint>true</preserveFixedJoint>
+    </gazebo>
+    <gazebo reference="robco_hand_tcp_joint">
+      <preserveFixedJoint>true</preserveFixedJoint>
+    </gazebo>
   </xacro:macro>
 </robot>

File: src/robco_description/ros2_control/robco.ros2_control.xacro (robot description, xacro)
@@ -7,5 +7,5 @@
       <hardware>
         <xacro:if value="${use_gazebo}">
-          <plugin>gz_ros2_control/GazeboSimSystem</plugin>
+          <plugin>gazebo_ros2_control/GazeboSystem</plugin>
         </xacro:if>
         <xacro:unless value="${use_gazebo}">

File: src/robco_description/urdf/handeye.xacro (robot description, xacro)
@@ -1,4 +1,5 @@
 <?xml version='1.0' encoding='utf-8'?>
 <robot xmlns:xacro="http://www.ros.org/wiki/xacro" name="robco">
+  <xacro:property name="description_package" value="$(find robco_description)" />
   <xacro:macro name="handeye"
     params="connected_to:='' ns:='' rpy:='0 0 0' xyz:='0 0 0' safety_distance:=0">
@@ -13,5 +14,5 @@
       <visual>
         <geometry>
-          <mesh filename="package://robco_description/meshes/handeye/d415_mount.stl" />
+          <mesh filename="file://${description_package}/meshes/handeye/d415_mount.stl" />
         </geometry>
         <material name="Gray">
@@ -31,4 +32,5 @@
         </geometry>
       </collision>
+      <xacro:inertials mesh_filename="handeye/d415_mount.stl"></xacro:inertials>
     </link>
     <joint name="${ns}_handeye_flange_joint" type="fixed">

File: src/robco_description/urdf/rg2.xacro (robot description, xacro)
@@ -3,4 +3,5 @@
   <xacro:property name="upper_gripper" value="0.5" />
   <xacro:property name="lower_gripper" value="0.77" />
+  <xacro:property name="description_package" value="$(find robco_description)" />
   <xacro:macro name="hand"
     params="connected_to:='' ns:='' rpy:='0 0 0' xyz:='0 0 0' safety_distance:=0">
@@ -15,5 +16,5 @@
       <visual>
         <geometry>
-          <mesh filename="package://robco_description/meshes/hand/quick_changer.stl" />
+          <mesh filename="file://${description_package}/meshes/hand/quick_changer.stl" />
         </geometry>
         <material name="Gray">
@@ -27,4 +28,5 @@
         </geometry>
       </collision>
+      <xacro:inertials mesh_filename="hand/quick_changer.stl"></xacro:inertials>
     </link>
     <joint name="${ns}_palmjoint" type="fixed">
@@ -36,5 +38,5 @@
       <visual>
         <geometry>
-          <mesh filename="package://robco_description/meshes/hand/rg2_palm.stl" />
+          <mesh filename="file://${description_package}/meshes/hand/rg2_palm.stl" />
         </geometry>
         <material name="Gray">
@@ -48,4 +50,5 @@
         </geometry>
       </collision>
+      <xacro:inertials mesh_filename="hand/rg2_palm.stl"></xacro:inertials>
     </link>
     <joint name="${ns}_left_finger_joint" type="revolute">
@@ -72,5 +75,5 @@
       <visual>
         <geometry>
-          <mesh filename="package://robco_description/meshes/hand/rg2_leftfinger.stl" />
+          <mesh filename="file://${description_package}/meshes/hand/rg2_leftfinger.stl" />
         </geometry>
         <material name="Gray">
@@ -78,4 +81,5 @@
         </material>
       </visual>
+      <xacro:inertials mesh_filename="hand/rg2_leftfinger.stl"></xacro:inertials>
     </link>
     <!-- MISSING COLLISION -->
@@ -83,5 +87,5 @@
       <visual>
         <geometry>
-          <mesh filename="package://robco_description/meshes/hand/rg2_rightfinger.stl" />
+          <mesh filename="file://${description_package}/meshes/hand/rg2_rightfinger.stl" />
         </geometry>
         <material name="Gray">
@@ -89,4 +93,5 @@
         </material>
       </visual>
+      <xacro:inertials mesh_filename="hand/rg2_rightfinger.stl"></xacro:inertials>
     </link>
     <joint name="${ns}_left_fingertip_joint" type="revolute">
@@ -114,5 +119,5 @@
       <visual>
         <geometry>
-          <mesh filename="package://robco_description/meshes/hand/rg2_leftfinger_tip.stl" />
+          <mesh filename="file://${description_package}/meshes/hand/rg2_leftfinger_tip.stl" />
         </geometry>
         <material name="Gray">
@@ -120,4 +125,5 @@
         </material>
       </visual>
+      <xacro:inertials mesh_filename="hand/rg2_leftfinger_tip.stl"></xacro:inertials>
     </link>
     <!-- MISSING COLLISION -->
@@ -125,5 +131,5 @@
       <visual>
         <geometry>
-          <mesh filename="package://robco_description/meshes/hand/rg2_rightfinger_tip.stl" />
+          <mesh filename="file://${description_package}/meshes/hand/rg2_rightfinger_tip.stl" />
         </geometry>
         <material name="Gray">
@@ -131,4 +137,5 @@
         </material>
       </visual>
+      <xacro:inertials mesh_filename="hand/rg2_rightfinger_tip.stl"></xacro:inertials>
     </link>
     <joint name="${ns}_hand_tcp_joint" type="fixed">

File: src/robco_description/urdf/robco.xacro (robot description, xacro)
@@ -1,6 +1,6 @@
 <?xml version="1.0"?>
 <robot xmlns:xacro="http://www.ros.org/wiki/xacro" name="robco">
-  <xacro:arg name="use_gazebo" default="false" />
-  <xacro:arg name="initial_positions_file" default="$(find robco_moveit_config)/config/initial_positions.yaml" />
+  <xacro:arg name="use_gazebo" default="true" />
+  <xacro:arg name="initial_positions_file" default="$(find robco_description)/config/initial_positions.yaml" />
   <!-- Import Robot macro -->
   <xacro:include filename="$(find robco_description)/urdf/robco_description.xacro" />
@@ -12,4 +12,5 @@
     <!-- Import Gazebo Classic definitions + plugin -->
     <xacro:include filename="$(find robco_description)/gazebo/robco_gazebo.xacro" />
+    <xacro:robco_gazebo/>
   </xacro:if>
 </robot>

File: src/robco_description/urdf/robco_modules_base.xacro (robot description, xacro)
@@ -1,10 +1,11 @@
 <?xml version="1.0"?>
 <robot xmlns:xacro="http://www.ros.org/wiki/xacro">
-    <xacro:property name="description_package" value="robco_description" />
+    <xacro:property name="description_package" value="$(find robco_description)" />
+    <xacro:include filename="$(find robco_description)/urdf/inertials.xacro"/>
     <xacro:macro name="robco_base_module" params="name mesh_filename tf_rpy tf_xyz next">
         <link name="${name}">
             <visual>
                 <geometry>
-                    <mesh filename="package://${description_package}/meshes/${mesh_filename}" />
+                    <mesh filename="file://${description_package}/meshes/${mesh_filename}" />
                 </geometry>
                 <material name="Gray">
@@ -14,7 +15,8 @@
             <collision>
                 <geometry>
-                    <mesh filename="package://${description_package}/meshes/${mesh_filename}" />
+                    <mesh filename="file://${description_package}/meshes/${mesh_filename}" />
                 </geometry>
             </collision>
+            <xacro:inertials mesh_filename="${mesh_filename}"/>
         </link>
         <xacro:if value="${next != ''}">
@@ -30,5 +32,5 @@
             <visual>
                 <geometry>
-                    <mesh filename="package://${description_package}/meshes/${mesh_filename}" />
+                    <mesh filename="file://${description_package}/meshes/${mesh_filename}" />
                 </geometry>
                 <material name="Gray">
@@ -38,7 +40,8 @@
             <collision>
                 <geometry>
-                    <mesh filename="package://${description_package}/meshes/${mesh_filename}" />
+                    <mesh filename="file://${description_package}/meshes/${mesh_filename}" />
                 </geometry>
             </collision>
+            <xacro:inertials mesh_filename="${mesh_filename}"/>
         </link>
         <xacro:if value="${next != ''}">
@@ -57,5 +60,5 @@
                 <geometry>
                     <mesh
-                        filename="package://${description_package}/meshes/${proximal_mesh_filename}" />
+                        filename="file://${description_package}/meshes/${proximal_mesh_filename}" />
                 </geometry>
                 <material name="Gray">
@@ -66,7 +69,8 @@
                 <geometry>
                     <mesh
-                        filename="package://${description_package}/meshes/${proximal_mesh_filename}" />
+                        filename="file://${description_package}/meshes/${proximal_mesh_filename}" />
                 </geometry>
             </collision>
+            <xacro:inertials mesh_filename="${proximal_mesh_filename}"/>
         </link>
         <joint name="${name}__${name}_shaft" type="fixed">
@@ -75,5 +79,7 @@
             <child link="${name}_shaft" />
         </joint>
-        <link name="${name}_shaft"></link>
+        <link name="${name}_shaft">
+            <xacro:inertials mesh_filename=""/>
+        </link>
         <joint name="${name}_joint" type="revolute">
             <origin rpy="${distal_tf_rpy}" xyz="${distal_tf_xyz}" />
@@ -86,5 +92,5 @@
             <visual>
                 <geometry>
-                    <mesh filename="package://${description_package}/meshes/${distal_mesh_filename}" />
+                    <mesh filename="file://${description_package}/meshes/${distal_mesh_filename}" />
                 </geometry>
                 <material name="Gray">
@@ -94,7 +100,8 @@
             <collision>
                 <geometry>
-                    <mesh filename="package://${description_package}/meshes/${distal_mesh_filename}" />
+                    <mesh filename="file://${description_package}/meshes/${distal_mesh_filename}" />
                 </geometry>
             </collision>
+            <xacro:inertials mesh_filename="${distal_mesh_filename}"/>
         </link>
         <xacro:if value="${next != ''}">
@@ -109,5 +116,5 @@
             <visual>
                 <geometry>
-                    <mesh filename="package://${description_package}/meshes/${mesh_filename}" />
+                    <mesh filename="file://${description_package}/meshes/${mesh_filename}" />
                 </geometry>
                 <material name="Red">
@@ -117,7 +124,8 @@
             <collision>
                 <geometry>
-                    <mesh filename="package://${description_package}/meshes/${mesh_filename}" />
+                    <mesh filename="file://${description_package}/meshes/${mesh_filename}" />
                 </geometry>
             </collision>
+            <xacro:inertials mesh_filename="${mesh_filename}"/>
         </link>
     </xacro:macro>
