Commit message: Got the validator to work!

File: src/robco_description/urdf/robco_description.xacro (robot description, xacro)
@@ -2,23 +2,19 @@
 <robot name="robco" xmlns:xacro="http://www.ros.org/wiki/xacro">
     <xacro:include filename="$(find robco_description)/urdf/robco_modules.xacro"/>
-    <link name="world" />
+    <link name="world"/>            <!-- Virtual link to fix the robot to the ground-->
     <joint name="world__base" type="fixed">
-                <origin rpy="0 0 0" xyz="0 0 0.132"/>
-                <parent link="world"/>
-                <child link="base"/>
+        <origin rpy="0 0 0" xyz="0 0 0.132"/>
+        <parent link="world"/>
+        <child link="base"/>
     </joint>
-    <xacro:robco_module_0106 name="base" next="drive1"/>
-    <xacro:robco_module_0088 name="drive1" next="drive2"/>
-    <xacro:robco_module_0089 name="drive2" next="link0"/>
-    <xacro:robco_module_0078 name="link0" next="drive3"/>
-    <xacro:robco_module_0085 name="drive3" next="drive4"/>
-    <xacro:robco_module_0085 name="drive4" next="link1"/>
-    <xacro:robco_module_0007 name="link1" next="drive5"/>
-    <xacro:robco_module_0085 name="drive5" next="drive6"/>
-    <xacro:robco_module_0085 name="drive6" next="effector"/>
-    <xacro:robco_module_0801 name="effector"/>
-    <!-- <xacro:include filename="$(find robco_description)/urdf/handeye.xacro"/>
-    <xacro:handeye ns="robco" rpy="0 0 0" connected_to="" safety_distance="0.00"/>
-    <xacro:include filename="$(find robco_description)/urdf/rg2.xacro"/>
-    <xacro:hand ns="robco" xyz="0 0 0" connected_to="robco_handeye_flange" safety_distance="0.0"/>  -->
+    <xacro:robco_module_0106 name="base" next="drive1"/>       <!-- Base module -->
+    <xacro:robco_module_0088 name="drive1" next="drive2"/>     <!-- Drive module -->
+    <xacro:robco_module_0089 name="drive2" next="link0"/>      <!-- Drive module -->
+    <xacro:robco_module_0078 name="link0" next="drive3"/>      <!-- Link module -->
+    <xacro:robco_module_0085 name="drive3" next="drive4"/>     <!-- Drive module -->
+    <xacro:robco_module_0085 name="drive4" next="link1"/>      <!-- Drive module -->
+    <xacro:robco_module_0007 name="link1" next="drive5"/>      <!-- Link module -->
+    <xacro:robco_module_0085 name="drive5" next="drive6"/>     <!-- Drive module -->
+    <xacro:robco_module_0085 name="drive6" next="effector"/>   <!-- Drive module -->
+    <xacro:robco_module_0801 name="effector"/>                 <!-- Effector module -->
 </robot>

File: src/robco_description/urdf/robco_modules_base.xacro (robot description, xacro)
@@ -1,7 +1,11 @@
 <?xml version="1.0"?>
 <robot xmlns="http://www.ros.org" xmlns:xacro="http://www.ros.org/wiki/xacro">
+    <!-- Gets resolved to the path to the robco_descrptions package -->
     <xacro:property name="description_package" value="$(find robco_description)" />
+    <!-- Base module -->
     <xacro:macro name="robco_base_module"
-        params="name mesh_filename tf_rpy tf_xyz proximal_mass proximal_ixx proximal_ixy proximal_ixz proximal_iyy proximal_iyz proximal_izz proximal_com_xyz next">
+        params="name mesh_filename tf_rpy tf_xyz proximal_mass
+                proximal_ixx proximal_ixy proximal_ixz proximal_iyy
+                proximal_iyz proximal_izz proximal_com_xyz next">
         <link name="${name}">
             <visual>
@@ -31,6 +35,9 @@
         </xacro:if>
     </xacro:macro>
+    <!-- Link module -->
     <xacro:macro name="robco_link_module"
-        params="name mesh_filename tf_rpy tf_xyz proximal_mass proximal_ixx proximal_ixy proximal_ixz proximal_iyy proximal_iyz proximal_izz proximal_com_xyz next">
+        params="name mesh_filename tf_rpy tf_xyz proximal_mass
+                proximal_ixx proximal_ixy proximal_ixz proximal_iyy
+                proximal_iyz proximal_izz proximal_com_xyz next">
         <link name="${name}">
             <visual>
@@ -46,7 +53,9 @@
             <inertial>
                 <mass value="${proximal_mass}" />
-                <inertia ixx="${proximal_ixx}" ixy="${proximal_ixy}" ixz="${proximal_ixz}"
-                    iyy="${proximal_iyy}" iyz="${proximal_iyz}"
-                    izz="${proximal_izz}" />
+                <inertia
+                    ixx="${proximal_ixx}" ixy="${proximal_ixy}"
+                    ixz="${proximal_ixz}" iyy="${proximal_iyy}"
+                    iyz="${proximal_iyz}" izz="${proximal_izz}"
+                />
                 <origin rpy="0 0 0" xyz="${proximal_com_xyz}" />
             </inertial>
@@ -60,6 +69,12 @@
         </xacro:if>
     </xacro:macro>
+    <!-- Drive module -->
     <xacro:macro name="robco_drive_module"
-        params="name proximal_mesh_filename distal_mesh_filename proximal_tf_rpy proximal_tf_xyz distal_tf_rpy distal_tf_xyz lim_lower:=-4.7124 lim_upper:=4.7124 proximal_mass proximal_ixx proximal_ixy proximal_ixz proximal_iyy proximal_iyz proximal_izz proximal_com_xyz distal_mass distal_ixx distal_ixy distal_ixz distal_iyy distal_iyz distal_izz distal_com_xyz next">
+        params="name proximal_mesh_filename distal_mesh_filename
+                proximal_tf_rpy proximal_tf_xyz distal_tf_rpy distal_tf_xyz
+                lim_lower:=-4.7124 lim_upper:=4.7124 proximal_mass proximal_ixx
+                proximal_ixy proximal_ixz proximal_iyy proximal_iyz proximal_izz
+                proximal_com_xyz distal_mass distal_ixx distal_ixy distal_ixz
+                distal_iyy distal_iyz distal_izz distal_com_xyz next">
         <!-- proximal link, calle ${name} to keep compatibility with next=... parameter -->
         <link name="${name}">
@@ -78,7 +93,9 @@
             <inertial>
                 <mass value="${proximal_mass}" />
-                <inertia ixx="${proximal_ixx}" ixy="${proximal_ixy}" ixz="${proximal_ixz}"
-                    iyy="${proximal_iyy}" iyz="${proximal_iyz}"
-                    izz="${proximal_izz}" />
+                <inertia
+                    ixx="${proximal_ixx}" ixy="${proximal_ixy}"
+                    ixz="${proximal_ixz}" iyy="${proximal_iyy}"
+                    iyz="${proximal_iyz}" izz="${proximal_izz}"
+                />
                 <origin rpy="0 0 0" xyz="${proximal_com_xyz}" />
             </inertial>
@@ -91,7 +108,7 @@
         <link name="${name}_shaft">
             <inertial>
-                <origin xyz="0 0 0" rpy="0 0 0"/>
-                <mass value="0.001"/>
-                <inertia ixx="0.0" ixy="0.0" ixz="0.0" iyy="0.0" iyz="0.0" izz="0.0"/>
+                <origin xyz="0 0 0" rpy="0 0 0" />
+                <mass value="0.001" />
+                <inertia ixx="0.0" ixy="0.0" ixz="0.0" iyy="0.0" iyz="0.0" izz="0.0" />
             </inertial>
         </link>
@@ -116,7 +133,9 @@
             <inertial>
                 <mass value="${distal_mass}" />
-                <inertia ixx="${distal_ixx}" ixy="${distal_ixy}" ixz="${distal_ixz}"
-                    iyy="${distal_iyy}" iyz="${distal_iyz}"
-                    izz="${distal_izz}" />
+                <inertia
+                    ixx="${distal_ixx}" ixy="${distal_ixy}"
+                    ixz="${distal_ixz}" iyy="${distal_iyy}"
+                    iyz="${distal_iyz}" izz="${distal_izz}"
+                />
                 <origin rpy="0 0 0" xyz="${distal_com_xyz}" />
             </inertial>
@@ -129,6 +148,9 @@
         </xacro:if>
     </xacro:macro>
+    <!-- Effector module -->
     <xacro:macro name="robco_end_effector"
-        params="name mesh_filename tf_rpy tf_xyz proximal_mass proximal_ixx proximal_ixy proximal_ixz proximal_iyy proximal_iyz proximal_izz proximal_com_xyz">
+        params="name mesh_filename tf_rpy tf_xyz proximal_mass
+                proximal_ixx proximal_ixy proximal_ixz proximal_iyy
+                proximal_iyz proximal_izz proximal_com_xyz">
         <link name="${name}">
             <visual>
@@ -144,7 +166,9 @@
             <inertial>
                 <mass value="${proximal_mass}" />
-                <inertia ixx="${proximal_ixx}" ixy="${proximal_ixy}" ixz="${proximal_ixz}"
-                    iyy="${proximal_iyy}" iyz="${proximal_iyz}"
-                    izz="${proximal_izz}" />
+                <inertia
+                    ixx="${proximal_ixx}" ixy="${proximal_ixy}"
+                    ixz="${proximal_ixz}" iyy="${proximal_iyy}"
+                    iyz="${proximal_iyz}" izz="${proximal_izz}"
+                />
                 <origin rpy="0 0 0" xyz="${proximal_com_xyz}" />
             </inertial>
