Commit message: Added validator, still needs tests

File: src/robco_description/urdf/robco_modules_base.xacro (robot description, xacro)
@@ -10,4 +10,9 @@
                 </geometry>
             </visual>
+            <collision>
+                <geometry>
+                    <mesh filename="file://${description_package}/meshes/${mesh_filename}" />
+                </geometry>
+            </collision>
             <inertial>
                 <mass value="${proximal_mass}" />
@@ -34,4 +39,9 @@
                 </geometry>
             </visual>
+            <collision>
+                <geometry>
+                    <mesh filename="file://${description_package}/meshes/${mesh_filename}" />
+                </geometry>
+            </collision>
             <inertial>
                 <mass value="${proximal_mass}" />
@@ -60,4 +70,10 @@
                 </geometry>
             </visual>
+            <collision>
+                <geometry>
+                    <mesh
+                        filename="file://${description_package}/meshes/${proximal_mesh_filename}" />
+                </geometry>
+            </collision>
             <inertial>
                 <mass value="${proximal_mass}" />
@@ -93,4 +109,9 @@
                 </geometry>
             </visual>
+            <collision>
+                <geometry>
+                    <mesh filename="file://${description_package}/meshes/${distal_mesh_filename}" />
+                </geometry>
+            </collision>
             <inertial>
                 <mass value="${distal_mass}" />
@@ -116,4 +137,9 @@
                 </geometry>
             </visual>
+            <collision>
+                <geometry>
+                    <mesh filename="file://${description_package}/meshes/${mesh_filename}" />
+                </geometry>
+            </collision>
             <inertial>
                 <mass value="${proximal_mass}" />

Commit message: Updated mainly all configs. Commit to make branch THESIS_DEADLINE possible

File: src/robco_description/urdf/robco_modules_base.xacro (robot description, xacro)
@@ -3,5 +3,5 @@
     <!-- Gets resolved to the path to the robco_descrptions package -->
     <xacro:property name="description_package" value="$(find robco_description)" />
-    <!-- Base module -->
+    <!-- Define materials -->
     <xacro:macro name="robco_base_module"
         params="name mesh_filename tf_rpy tf_xyz proximal_mass
@@ -13,4 +13,7 @@
                     <mesh filename="file://${description_package}/meshes/${mesh_filename}" />
                 </geometry>
+                <material name="White">
+                  <color rgba="1.0 1.0 1.0 1.0"/>
+                </material>
             </visual>
             <collision>
@@ -45,4 +48,7 @@
                     <mesh filename="file://${description_package}/meshes/${mesh_filename}" />
                 </geometry>
+                <material name="White">
+                  <color rgba="1.0 1.0 1.0 1.0"/>
+                </material>
             </visual>
             <collision>
@@ -84,4 +90,7 @@
                         filename="file://${description_package}/meshes/${proximal_mesh_filename}" />
                 </geometry>
+                <material name="White">
+                  <color rgba="1.0 1.0 1.0 1.0"/>
+                </material>
             </visual>
             <collision>
@@ -125,4 +134,7 @@
                     <mesh filename="file://${description_package}/meshes/${distal_mesh_filename}" />
                 </geometry>
+                <material name="White">
+                  <color rgba="1.0 1.0 1.0 1.0"/>
+                </material>
             </visual>
             <collision>
@@ -158,4 +170,7 @@
                     <mesh filename="file://${description_package}/meshes/${mesh_filename}" />
                 </geometry>
+                <material name="White">
+                  <color rgba="1.0 1.0 1.0 1.0"/>
+                </material>
             </visual>
             <collision>
